Commit message: fix: Rotate laser on pi/2  in order to look in front

File: my_robot/urdf/my_robot.xacro (robot description, xacro)
@@ -222,5 +222,5 @@
         <inertial>
         <mass value="1e-1"/>
-            <origin xyz="0 0 0" rpy="0 0 0"/>
+            <origin xyz="0 0 0" rpy="0 0 1.570796"/>
             <box_inertia sizeX="0.05" sizeY="0.05" sizeZ="0.05" mass="0.1"/>
             <inertia ixx="1e-6" ixy="0" ixz="0" iyy="1e-6" iyz="0" izz="1e-6"/>
